File: raspberry-pi-hat/unisonht.kicad_sch (KiCad schematic)
At the start: 20 parts, among them J1 Raspberry_Pi_2_3, J2 IROUT, J3 IROUT, J4 IROUT, J5 IROUT, Q1 2N7002E, U1 MCP3204

Commit message: initial schematic
Parts:
- added C3: 0.1uF, symbol Device:C
- added D3: POWER, LED_SMD:LED_0805_2012Metric, symbol Device:LED
- added J10: FRONT, symbol Connector_Generic:Conn_02x05_Odd_Even
- added J11: Conn_01x08, Connector_PinHeader_2.54mm:PinHeader_1x08_P2.54mm_Vertical, symbol Connector_Generic:Conn_01x08
- added J6: ADC, Connector_PinHeader_2.54mm:PinHeader_1x08_P2.54mm_Vertical, symbol Connector:Conn_01x08_Pin
- added J7: FAN, Connector_PinHeader_2.54mm:PinHeader_1x02_P2.54mm_Vertical, symbol Connector:Conn_01x02_Pin
- added J8: IROUT, Connector_PinHeader_2.54mm:PinHeader_2x02_P2.54mm_Vertical, symbol Connector_Generic:Conn_02x02_Odd_Even
- added J9: IRIN, symbol Connector_Generic:Conn_02x03_Odd_Even
- added Q2: BSS84, Package_TO_SOT_SMD:SOT-23, symbol Transistor_FET:BSS84
- added R10, R11, R12, R13: 100k, Resistor_SMD:R_0805_2012Metric, symbol Device:R
- added R14: 180, Resistor_SMD:R_0805_2012Metric, symbol Device:R
- added R15: 10K, Resistor_SMD:R_0805_2012Metric, symbol Device:R
- D1: value LED -> IROUT
- D2: value LED -> IRIN
- J3: value IROUT -> IRIN
Connections:
- net +3.3V: now also C3.1, D3.2 (A), J10.1 (Pin_1), J11.1 (Pin_1), J6.2 (Pin_2), J8.1 (Pin_1), J9.1 (Pin_1), Q2.3 (D), R15.2
- net +5V: now also J10.2 (Pin_2), J11.2 (Pin_2), J6.1 (Pin_1), J7.1 (Pin_1)
- net GND: now also C3.2, J10.9 (Pin_9), J11.8 (Pin_8), J6.8 (Pin_8), J7.2 (Pin_2), J9.5 (Pin_5), R12.1, R13.1, R14.1; no longer U1.3 (CH2), U1.4 (CH3)
- net IRIN: now also J10.4 (Pin_4), J9.3 (Pin_3), Q2.1 (G), R15.1; no longer D2.2 (A)
- net IROUT: now also J10.6 (Pin_6)
- net VMID: now also J6.7 (Pin_7), R10.1, R11.1
- net ADCCH1: now reaches J5.T, U1.2 (CH1)
- net ADCCH1: now also J6.4 (Pin_4), R10.2
- net at J3.R: now also J9.4 (Pin_4)
- net at J3.S: now also J9.6 (Pin_6)
- net at J3.T: now also J9.2 (Pin_2)
- net IROUT_DRAIN: now reaches Q1.3 (D), R3.1, R4.1
- net IROUT_DRAIN: now also J10.5 (Pin_5)
- net ADCCH0: now reaches J4.T, U1.1 (CH0)
- net ADCCH0: now also J6.3 (Pin_3), R11.2
- net RXD: now reaches J1.10 (GPIO15/RXD)
- net RXD: now also J10.8 (Pin_8), J11.4 (Pin_4)
- net GPIO12: now reaches J1.32 (PWM0/GPIO12)
- net GPIO12: now also J10.10 (Pin_10), J11.5 (Pin_5)
- net GPIO13: now reaches J1.33 (PWM1/GPIO13)
- net GPIO13: now also J11.6 (Pin_6)
- net GPIO16: now reaches J1.36 (GPIO16)
- net GPIO16: now also J11.7 (Pin_7)
- net TXD: now reaches J1.8 (GPIO14/TXD)
- net TXD: now also J10.7 (Pin_7), J11.3 (Pin_3)
- net at J2.S: now also J8.4 (Pin_4)
- net at J2.T: now also J8.2 (Pin_2)
- net at R4.2: now also J8.3 (Pin_3)
- new net: D3.1 (K), R14.2
- new net ADCCH2: J6.5 (Pin_5), R12.2, U1.3 (CH2)
- new net ADCCH3: J6.6 (Pin_6), R13.2, U1.4 (CH3)
- new net IRIN_DRAIN: D2.2 (A), J10.3 (Pin_3), Q2.2 (S)
- no-connect marks 22 -> 20
Other:
- moved on the sheet: C1, C2, D1, D2, J2, J3, J4, J5, Q1, R1, R2, R3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
